File: comp_and_pwr_pcb.kicad_pcb (KiCad board)
At the start: 4 copper layers, 50 x 88.5 mm, 145 parts, among them IC1 TPS5430MDDAREP, IC3 LTC4415EDHC#TRPBF, IC4 TPS259531DSGR, IC5 BMP388, IC6 W25Q32JVSSIQ, J1 USB4216-03-A, J10 Conn_01x02, J11 Conn_Coaxial, J12 Conn_Coaxial, J2 BATTERY_CONN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

Commit message: Update drc for aisler, update .gitignore
Routing:
- net /CAMERA_SWITCH: track 60.2 -> 60.8 mm
Other:
- board text added: "2025"
- board text added: "RTU HPR"
